File: Kicad/Scout_radio/ScoutAM.kicad_pcb (KiCad board)
At the start: 2 copper layers, 55 x 100 mm, 92 parts, among them J1 Conn_01x07, J2 Conn_01x02, J3 PJ-342, J4 Conn_Coaxial, J5 Conn_01x02, Q1 AO3401A, Q2 2N7002, SW1 TC-6610-5-260G, SW2 TC-6610-5-260G, SW3 TC-6610-5-260G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

Commit message: Updated README.md
Parts:
- SW1, SW2, SW3, SW4, SW5, SW6: value TC-6610-5-260G -> B3FS; footprint Button_Switch_SMD:SW_Push_1P1T_NO_6x6mm_H9.5mm -> Scout:SW_Push_1P1T_NO_6x6mm_H9.5mm
Changed lines of the file:
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@@
 			)
 		)
+		(property "Sim.Enable" ""
+			(at 0 0 180)
+			(unlocked yes)
+			(layer "F.Fab")
+			(hide yes)
+			(effects
+				(font
+					(size 1 1)
+					(thickness 0.15)
+				)
+			)
+		)
 		(property ki_fp_filters "R_*")
 		(sheetname "Root")
@@
 			)
 		)
+		(property "Sim.Enable" ""
+			(at 0 0 180)
+			(unlocked yes)
+			(layer "F.Fab")
+			(hide yes)
+			(effects
+				(font
+					(size 1 1)
+					(thickness 0.15)
+				)
+			)
+		)
 		(property ki_fp_filters "R_*")
 		(sheetname "Root")
@@
 		)
 	)
-	(footprint "Button_Switch_SMD:SW_Push_1P1T_NO_6x6mm_H9.5mm"
+	(footprint "Scout:SW_Push_1P1T_NO_6x6mm_H9.5mm"
 		(layer "F.Cu")
 		(at 114.635 136.32)
@@
 			)
 		)
-		(property "Value" "TC-6610-5-260G"
+		(property "Value" "B3FS"
 			(at 0 4.15 0)
 			(layer "F.Fab")
@@
 			)
 		)
-		(property "Footprint" "Button_Switch_SMD:SW_Push_1P1T_NO_6x6mm_H9.5mm"
+		(property "Footprint" "Scout:SW_Push_1P1T_NO_6x6mm_H9.5mm"
 			(at 0 0 0)
 			(unlocked yes)
@@
 			)
 		)
-		(property "Sim.Enable" ""
+		(property "LCSC" ""
 			(at 0 0 0)
 			(unlocked yes)
@@
 			)
 		)
-		(property "LCSC" ""
+		(property "Sim.Enable" ""
 			(at 0 0 0)
 			(unlocked yes)
@@
 		)
 	)
-	(footprint "Button_Switch_SMD:SW_Push_1P1T_NO_6x6mm_H9.5mm"
+	(footprint "Scout:SW_Push_1P1T_NO_6x6mm_H9.5mm"
 		(layer "F.Cu")
 		(at 96.88 145.36)
@@
 			)
 		)
-		(property "Value" "TC-6610-5-260G"
+		(property "Value" "B3FS"
 			(at 0 4.15 0)
 			(layer "F.Fab")
@@
 			)
 		)
-		(property "Footprint" "Button_Switch_SMD:SW_Push_1P1T_NO_6x6mm_H9.5mm"
+		(property "Footprint" "Scout:SW_Push_1P1T_NO_6x6mm_H9.5mm"
 			(at 0 0 0)
 			(unlocked yes)
@@
 			)
 		)
-		(property "Sim.Enable" ""
+		(property "LCSC" ""
 			(at 0 0 0)
 			(unlocked yes)
@@
 			)
 		)
-		(property "LCSC" ""
+		(property "Sim.Enable" ""
 			(at 0 0 0)
 			(unlocked yes)
@@
 		)
 	)
-	(footprint "Button_Switch_SMD:SW_Push_1P1T_NO_6x6mm_H9.5mm"
+	(footprint "Scout:SW_Push_1P1T_NO_6x6mm_H9.5mm"
 		(layer "F.Cu")
 		(at 80.085 145.36)
@@
 			)
 		)
-		(property "Value" "TC-6610-5-260G"
+		(property "Value" "B3FS"
 			(at 0 4.15 0)
 			(layer "F.Fab")
@@
 			)
 		)
-		(property "Footprint" "Button_Switch_SMD:SW_Push_1P1T_NO_6x6mm_H9.5mm"
+		(property "Footprint" "Scout:SW_Push_1P1T_NO_6x6mm_H9.5mm"
 			(at 0 0 0)
 			(unlocked yes)
@@
 			)
 		)
-		(property "Sim.Enable" ""
+		(property "LCSC" ""
 			(at 0 0 0)
 			(unlocked yes)
@@
 			)
 		)
-		(property "LCSC" ""
+		(property "Sim.Enable" ""
 			(at 0 0 0)
 			(unlocked yes)
@@
 		)
 	)
-	(footprint "Button_Switch_SMD:SW_Push_1P1T_NO_6x6mm_H9.5mm"
+	(footprint "Scout:SW_Push_1P1T_NO_6x6mm_H9.5mm"
 		(layer "F.Cu")
 		(at 97.215 136.43)
@@
 			)
 		)
-		(property "Value" "TC-6610-5-260G"
+		(property "Value" "B3FS"
 			(at 0 4.15 0)
 			(layer "F.Fab")
@@
 			)
 		)
-		(property "Footprint" "Button_Switch_SMD:SW_Push_1P1T_NO_6x6mm_H9.5mm"
+		(property "Footprint" "Scout:SW_Push_1P1T_NO_6x6mm_H9.5mm"
 			(at 0 0 0)
 			(unlocked yes)
@@
 			)
 		)
-		(property "Sim.Enable" ""
+		(property "LCSC" ""
 			(at 0 0 0)
 			(unlocked yes)
@@
 			)
 		)
-		(property "LCSC" ""
+		(property "Sim.Enable" ""
 			(at 0 0 0)
 			(unlocked yes)
@@
 		)
 	)
-	(footprint "Button_Switch_SMD:SW_Push_1P1T_NO_6x6mm_H9.5mm"
+	(footprint "Scout:SW_Push_1P1T_NO_6x6mm_H9.5mm"
 		(layer "F.Cu")
 		(at 80.185 136.61)
@@
 			)
 		)
-		(property "Value" "TC-6610-5-260G"
+		(property "Value" "B3FS"
 			(at 0 4.15 0)
 			(layer "F.Fab")
@@
 			)
 		)
-		(property "Footprint" "Button_Switch_SMD:SW_Push_1P1T_NO_6x6mm_H9.5mm"
+		(property "Footprint" "Scout:SW_Push_1P1T_NO_6x6mm_H9.5mm"
 			(at 0 0 0)
 			(unlocked yes)
@@
 			)
 		)
-		(property "Sim.Enable" ""
+		(property "LCSC" ""
 			(at 0 0 0)
 			(unlocked yes)
@@
 			)
 		)
-		(property "LCSC" ""
+		(property "Sim.Enable" ""
 			(at 0 0 0)
 			(unlocked yes)
@@
 		)
 	)
-	(footprint "Button_Switch_SMD:SW_Push_1P1T_NO_6x6mm_H9.5mm"
+	(footprint "Scout:SW_Push_1P1T_NO_6x6mm_H9.5mm"
 		(layer "F.Cu")
 		(at 114.675 145.32)
@@
 			)
 		)
-		(property "Value" "TC-6610-5-260G"
+		(property "Value" "B3FS"
 			(at 0 4.15 0)
 			(layer "F.Fab")
@@
 			)
 		)
-		(property "Footprint" "Button_Switch_SMD:SW_Push_1P1T_NO_6x6mm_H9.5mm"
+		(property "Footprint" "Scout:SW_Push_1P1T_NO_6x6mm_H9.5mm"
 			(at 0 0 0)
 			(unlocked yes)
@@
 			)
 		)
-		(property "Sim.Enable" ""
+		(property "LCSC" ""
 			(at 0 0 0)
 			(unlocked yes)
@@
 			)
 		)
-		(property "LCSC" ""
+		(property "Sim.Enable" ""
 			(at 0 0 0)
 			(unlocked yes)
